File: hw/pcb/TrueStrike56.kicad_sch (KiCad schematic)
At the start: 198 parts, among them SW1 SW_Push, U1 ProMicro, U10 4053, U2 74HC4051, U3 74HC4051, U4 74HC4051, U5 74HC4051, U6 74HC4051, U7 74HC4051, U8 74HC4051, U9 74AHCT125

Commit message: Add logo+model name+rev #, set LCSC Part # for PCBA order
Parts:
- Brd1, U1: now left out of the parts list
- C1, C10, C11, C12, C13, C14, C15, C16, C17, C18, C19, C2, C20, C21, C22, C23, C24, C25, C26, C27, C28, C29, C3, C30, C31, C32, C33, C34, C35, C36, C37, C38, C39, C4, C40, C41, C42, C43, C44, C45, C46, C47, C48, C49, C5, C50, C51, C52, C53, C54, C55, C56, C57, C58, C59, C6, C60, C61, C62, C63, C64, C65, C66, C67, C68, C69, C7, C70, C71, C72, C73, C74, C8, C9: LCSC Part # (none) -> C28233
- D1, D10, D11, D12, D13, D14, D15, D16, D17, D18, D19, D2, D20, D21, D22, D23, D24, D25, D26, D27, D28, D29, D3, D30, D31, D32, D33, D34, D35, D36, D37, D38, D39, D4, D40, D41, D42, D43, D44, D45, D46, D47, D48, D49, D5, D50, D51, D52, D53, D54, D55, D56, D6, D7, D8, D9: LCSC Part # (none) -> C5149201
- S1, S10, S11, S12, S13, S14, S15, S16, S17, S18, S19, S2, S20, S21, S22, S23, S24, S25, S26, S27, S28, S29, S3, S30, S31, S32, S33, S34, S35, S36, S37, S38, S39, S4, S40, S41, S42, S43, S44, S45, S46, S47, S48, S49, S5, S50, S51, S52, S53, S54, S55, S56, S6, S7, S8, S9: LCSC Part # (none) -> C126669
- U10: LCSC Part # (none) -> C5647
- U2, U3, U4, U5, U6, U7, U8: LCSC Part # (none) -> C85220
- U9: LCSC Part # (none) -> C155176

Commit message: Update PCB and production files for PCBA
Changed RESET tactile switch to JLCPCB PCBA compatible part
Parts:
- SW1: footprint Button_Switch_SMD:SW_Tactile_SPST_NO_Straight_CK_PTS636Sx25SMTRLFS -> Button_Switch_SMD:SW_Push_1P1T_XKB_TS-1187A; LCSC Part # (none) -> C318884
Changed lines of the file:
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@@
 			)
 		)
-		(property "Footprint" "Button_Switch_SMD:SW_Tactile_SPST_NO_Straight_CK_PTS636Sx25SMTRLFS"
+		(property "Footprint" "Button_Switch_SMD:SW_Push_1P1T_XKB_TS-1187A"
 			(at 293.37 283.21 0)
 			(effects
@@
 			)
 		)
-		(property "LCSC Part #" ""
+		(property "LCSC Part #" "C318884"
 			(at 293.37 288.29 0)
 			(effects
