File: hw/pcb/TrueStrike56.kicad_pcb (KiCad board)
At the start: 2 copper layers, 278.9 x 138.4 mm, 211 parts, among them SW1 SW_Push, U1 ProMicro, U10 4053, U2 74HC4051, U3 74HC4051, U4 74HC4051, U5 74HC4051, U6 74HC4051, U7 74HC4051, U8 74HC4051, U9 74AHCT125

Commit message: Update HE switch footprint to have the correct side
Parts:
- S1, S10, S11, S12, S13, S14, S15, S16, S17, S18, S19, S2, S20, S21, S22, S23, S24, S25, S26, S27, S28, S29, S3, S30, S31, S32, S33, S34, S35, S36, S37, S38, S39, S4, S40, S41, S42, S43, S44, S45, S46, S47, S48, S49, S5, S50, S51, S52, S53, S54, S55, S56, S6, S7, S8, S9: moved to B.Cu
- turned S1 to 165 degrees
- turned S10 to 165 degrees
- turned S11 to 165 degrees
- turned S12 to 165 degrees
- turned S13 to 165 degrees
- turned S14 to 165 degrees
- turned S15 to 165 degrees
- turned S16 to 165 degrees
- turned S17 to 165 degrees
- turned S18 to 165 degrees
- turned S19 to 165 degrees
- turned S2 to 165 degrees
- turned S20 to 165 degrees
- turned S21 to 165 degrees
- turned S22 to 165 degrees
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